File: design_files/ASD2831.brd (EAGLE design)
At the start: 22.5 x 22.5 mm, 10 parts, among them J1 DF12-32-DP, J2 DF12-32-DS, U1 DS1339, Y1 300-8739-1-ND

Commit message: update format
Parts:
- R4: value (none) -> 0.0
Other:
- board size 22.5 x 22.5 mm -> 20 x 20 mm
- board text added: "TinyCircuits.com"
- board text removed: "Tiny-Circuits.com"
Changed lines of the file:
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@@
 <setting verticaltext="up"/>
 </settings>
-<grid distance="2" unitdist="mil" unit="mm" style="lines" multiple="1" display="yes" altdistance="1" altunitdist="mil" altunit="mil"/>
+<grid distance="0.1" unitdist="mm" unit="mm" style="lines" multiple="1" display="yes" altdistance="1" altunitdist="mil" altunit="mil"/>
 <layers>
 <layer number="1" name="Top" color="4" fill="1" visible="yes" active="yes"/>
@@
 <text x="44.986825" y="1.7714" size="0.889" layer="48">AS-PCB-ASD2831</text>
 <text x="67.3810375" y="1.6952" size="0.889" layer="48">4</text>
-<text x="21.6862" y="18.83995" size="0.635" layer="21" rot="R180">Tiny-Circuits.com</text>
+<text x="21.6862" y="18.83995" size="0.635" layer="21" rot="R180">TinyCircuits.com</text>
 <wire x1="10" y1="30" x2="30" y2="30" width="0.0254" layer="20"/>
 <wire x1="30" y1="30" x2="30" y2="10" width="0.0254" layer="20"/>
@@
 <hole x="11.5" y="11.5" drill="1.5"/>
 <dimension x1="10" y1="30" x2="10" y2="10" x3="7" y3="20" layer="48"/>
-<wire x1="31.27" y1="31.27" x2="31.27" y2="21.73" width="2.54" layer="46"/>
-<wire x1="31.27" y1="18.27" x2="31.27" y2="8.73" width="2.54" layer="46"/>
-<wire x1="31.27" y1="8.73" x2="21.73" y2="8.73" width="2.54" layer="46"/>
-<wire x1="18.27" y1="8.73" x2="8.73" y2="8.73" width="2.54" layer="46"/>
-<wire x1="8.73" y1="8.73" x2="8.73" y2="18.27" width="2.54" layer="46"/>
-<wire x1="8.73" y1="21.73" x2="8.73" y2="31.27" width="2.54" layer="46"/>
-<wire x1="8.73" y1="31.27" x2="18.27" y2="31.27" width="2.54" layer="46"/>
-<wire x1="21.73" y1="31.27" x2="31.27" y2="31.27" width="2.54" layer="46"/>
 <text x="40.3098" y="14.837396875" size="0.4572" layer="48" ratio="10">Released under the Creative Commons Attribution Share-Alike 3.0 License</text>
 <text x="40.3098" y="14.075396875" size="0.4572" layer="48" ratio="10">http://creativecommons.org/licenses/by-sa/3.0</text>
@@
 <rectangle x1="17.853659375" y1="28.0924" x2="18.072096875" y2="28.097475" layer="22"/>
 <rectangle x1="17.879059375" y1="28.097478125" x2="18.041615625" y2="28.102559375" layer="22"/>
-<text x="14.889078125" y="23.442215625" size="0.762" layer="22" rot="MR180">Tiny-Circuits.com</text>
+<text x="14.889078125" y="23.442215625" size="0.762" layer="22" rot="MR180">TinyCircuits.com</text>
 <text x="15.399721875" y="22.0550875" size="0.762" layer="22" rot="MR180">ASD2831- Rev4</text>
 <text x="15.167103125" y="20.89656875" size="0.762" layer="22" rot="MR180">Real Time Clock</text>
@@
 <attribute name="PARTNO" value="AS-ITM-00183" x="17.145" y="27.051" size="1.778" layer="27" display="off"/>
 </element>
-<element name="R4" library="tinycircuits" package="0402_SHORT" value="" x="15.3162" y="20.32" rot="R180">
+<element name="R4" library="tinycircuits" package="0402_SHORT" value="0.0" x="15.3162" y="20.32" rot="R180">
 <attribute name="VALUE" value="SHORT" x="15.3162" y="20.32" size="1.778" layer="27" rot="R180" display="off"/>
+<attribute name="PARTNO" value="AS-ITM-00076" x="15.3162" y="20.32" size="1.778" layer="27" rot="R180" display="off"/>
 </element>
 <element name="R5" library="tinycircuits" package="0402" value="0.0" x="15.367" y="19.431" rot="R180">
