File: design_files/ASD2831.sch (EAGLE design)
At the start: 9 parts, among them J1 DF12-32-DP, J2 DF12-32-DS, U1 DS1339, Y1 300-8739-1-ND

Commit message: update format
Parts:
- R4: value (none) -> 0.0
Other:
- note added: "Hand Populated: Y1"
- note added: "Hand Soldered: B1"
- note added: "Non Populated: R4, R5"
- note added: "Notes: Battery attached with Locktite 382 after reflow and hand soldered."
- note added: "Variant: Standard - R"
Changed lines of the file:
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@@
 <attribute name="VALUE" value="CM200C-32.768KDZBT"/>
 </part>
-<part name="R4" library="tinycircuits" deviceset="AS-ITM-00076" device="0402_SHORT"/>
+<part name="R4" library="tinycircuits" deviceset="AS-ITM-00076" device="0402_SHORT" value="0.0"/>
 <part name="R5" library="tinycircuits" deviceset="AS-ITM-00076" device="" value="0.0"/>
 <part name="C1" library="tinycircuits" deviceset="AS-ITM-00008" device="" value="0.1uF"/>
@@
 <text x="45.72" y="20.32" size="3.048" layer="91">Original Arduino Uno Design by Team Arduino</text>
 <text x="142.24" y="193.548" size="3.81" layer="94" font="vector">Maxim DS1339</text>
+<text x="50.8" y="55.88" size="1.778" layer="97">Non Populated: R4, R5</text>
+<text x="50.8" y="53.34" size="1.778" layer="97">Hand Populated: Y1</text>
+<text x="50.8" y="50.8" size="1.778" layer="97">Hand Soldered: B1</text>
+<text x="50.8" y="48.26" size="1.778" layer="97">Notes: Battery attached with Locktite 382 after reflow and hand soldered.</text>
+<text x="50.8" y="58.42" size="1.778" layer="97">Variant: Standard - R</text>
 </plain>
 <instances>
